File: Smart-Switch.kicad_pcb (KiCad board)
At the start: 2 copper layers, 13 parts, among them J1 Conn_WallSocket_Earth, K1 FINDER-40.11, P1 Conn_WallPlug_Earth, Q1 Q_NPN_EBC, U1 L78L33_TO92, U2 ESP-12E

Commit message: 1
Routing:
- net GND: track 0.00 -> 35.9 mm
- added copper zone on F.Cu, net GND
- added copper zone on F.Cu, net Net-(J1-Pad1)
- added copper zone on F.Cu, net Net-(J1-Pad2)
- added copper zone on F.Cu, net Net-(J1-Pad3)
- added copper zone on F.Cu, net Net-(K1-Pad14)
Other:
- net class Default: clearance 0.2 -> 1
- rule trace_clearance: 0.2 -> 1
- board text added: "E"
- board text added: "L"
- board text added: "N"
